File: schematic/Spotify Display.kicad_sch (KiCad schematic)
At the start: 6 parts, among them J1 LOLIN_C3_MINI_LEFT, J2 LOLIN_C3_MINI_RIGHT, J3 ST7735, SW1 SW_Push, SW2 SW_Push, SW3 SW_Push

Commit message: Update schematic
Parts:
- added D1: LED, symbol Device:LED
- added R1: 150R, symbol Device:R
- added SW4: SW_Push, symbol Switch:SW_Push
Connections:
- net GND: now also D1.1 (K), SW4.2
- net at J2.1 (GPIO21_TX): now also R1.1
- net SW4: now reaches J2.4 (GPIO8)
- net SW4: now also SW4.1
- new net LED: D1.2 (A), R1.2
- no-connect marks 6 -> 4
